File: doc/EaglePCB/ESP8266-DS18B20.brd (EAGLE design)
At the start: 72.1 x 40.6 mm, 10 parts, among them IC2 DS1820, IC3 LM340S

Commit message: small fixes
Parts:
- R1: value 10k -> 1k
Changed lines of the file:
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@@
 <element name="IC2" library="DS1820" package="TO-92" value="DS1820" x="62.23" y="68.58"/>
 <element name="IC3" library="linear" package="SOT223" value="LM340S" x="44.45" y="53.34" rot="MR180"/>
-<element name="R1" library="resistor" package="0207/12" value="10k" x="31.75" y="43.18"/>
+<element name="R1" library="resistor" package="0207/12" value="1k" x="31.75" y="43.18"/>
 <element name="R2" library="resistor" package="0207/12" value="4.7k" x="63.5" y="49.53" rot="R90"/>
 <element name="RST" library="switch-omron" package="B3F-10XX" value="" x="29.21" y="53.34">
