File: doc/EaglePCB/esp8266-DS18B20.sch (EAGLE design)
At the start: 10 parts, among them IC2 DS1820, IC3 LM340S

Commit message: small fixes
Parts:
- R1: value 10k -> 1k
Changed lines of the file:
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@@
 <part name="D2" library="diode" deviceset="1N4004" device=""/>
 <part name="C2" library="rcl" deviceset="CPOL-EU" device="E2.5-5" value="100uF"/>
-<part name="R1" library="resistor" deviceset="R-EU_" device="0207/12" value="10k"/>
+<part name="R1" library="resistor" deviceset="R-EU_" device="0207/12" value="1k"/>
 <part name="R2" library="resistor" deviceset="R-EU_" device="0207/12" value="4.7k"/>
 <part name="C1" library="rcl" deviceset="CPOL-EU" device="E2.5-5" value="100uf"/>
